Commit message: xacro and luanch editing

File: urdf/ropot.xacro (robot description, xacro)
@@ -1,6 +1,14 @@
-<?xml version="1.0"?>
 <?xml version='1.0'?>
 <robot name="box_ropot" xmlns:xacro="http://www.ros.org/wiki/xacro">
-<xacro:include filename="$(find mybot_description)/urdf/plugin.gazebo" />
+<xacro:include filename="$(find urdf_trial_discription)/urdf/plugin.gazebo" />
+<link name="base_link">
+</link>
+    <joint name="base_link_joint" type="fixed">
+        <origin xyz="0.0 0.0 0.0" rpy="0.0 0.0 0.0"/>
+        <parent link="base_link"/>
+        <child link="base_plate"/>
+        <axis xyz="0.0 0.0 0.0"/>
+        <limit lower="0.0" upper="0.0" effort="0.0" velocity="0.0"/>
+    </joint>
 <link name="base_plate">
     <inertial>
@@ -10,5 +18,5 @@
     </inertial>
     <visual name="plate_visual">
-        <origin xyz="0.0 0.04 0.0" rpy="0.0 0.0 0.0"/>
+        <origin xyz="0.0 0.0 0.05" rpy="1.5707 0.0 0.0"/>
         <geometry>
             <box size=".2 .026 .3"/>
@@ -20,5 +28,5 @@
     </visual>
     <collision>
-        <origin xyz="0.0 0.04 0.0" rpy="0.0 0.0 0.0"/>
+        <origin xyz="0.0 0.0 0.0" rpy="0.0 0.0 0.0"/>
         <geometry>
             <box size=".2 .026 .3"/>
@@ -33,5 +41,5 @@
     </inertial>
     <visual name="upper_plate_visual">
-        <origin xyz="0.0 0.13 0.0" rpy="0.0 0.0 0.0"/>
+        <origin xyz="0.0 0.0 0.09" rpy="1.5707 0.0 0.0"/>
         <geometry>
             <box size=".2 .019 .3"/>
@@ -43,5 +51,5 @@
     </visual>
     <collision>
-        <origin xyz="0.0 0.13 0.0" rpy="0.0 0.0 0.0"/>
+        <origin xyz="0.0 0.0 0.09" rpy="1.5707 0.0 0.0"/>
         <geometry>
             <box size=".2 .019 .3"/>
@@ -49,14 +57,21 @@
     </collision>
 </link>
+<joint name="upper_plate_joint" type="fixed">
+    <origin xyz="0.0 0.0 0.05" rpy="0 0.0 0.0"/>
+    <parent link="base_link"/>
+    <child link="upper_plate"/>
+    <axis xyz="0.0 0.0 0.0"/>
+    <limit lower="0.0" upper="0.0" effort="0.0" velocity="0.0"/>
+</joint>
 <link name="left__back_wheel">
     <inertial>
-        <origin xyz="0.0 0.0 0.0" rpy="0 0.0 0.0"/>
-        <mass value="0.0"/>
+        <origin xyz="0.11 0.1 0.0" rpy="0 0.0 0"/>
+        <mass value="0.3"/>
         <inertia ixx="0.0" ixy="0.0" ixz="0.0" iyy="0.0" iyz="0.0" izz="0.0"/>
     </inertial>
     <visual name="left__back_wheel_visual">
-        <origin xyz="0.11 0.04 0.07" rpy="0 1.5707 0.0"/>
-        <geometry>
-            <cylinder radius="0.05" length="0.02"/>
+        <origin xyz="0.0 0.0 0.0" rpy="0 1.5707 1.5707"/>
+        <geometry>
+            <cylinder radius="0.04" length="0.02"/>
         </geometry>
         <material name="">
@@ -66,12 +81,12 @@
     </visual>
     <collision>
-        <origin xyz="0.11 0.04 0.07" rpy="0 1.5707 0.0"/>
-        <geometry>
-             <cylinder radius="0.05" length="0.02"/>
-        </geometry>
-    </collision>
-</link>
-<joint name="left__back_wheel_joint" type="revolute">
-    <origin xyz="0.11 0.04 0.07" rpy="0.0 0.0 0.0"/>
+        <origin xyz="0.0 0.0 0.0" rpy="0 0 0.0"/>
+        <geometry>
+             <cylinder radius="0.04" length="0.02"/>
+        </geometry>
+    </collision>
+</link>
+<joint name="left__back_wheel_joint" type="continuous">
+    <origin xyz="-0.11 -0.06 0.04" rpy="0 0.0 -1.57"/>
     <parent link="base_plate"/>
     <child link="left__back_wheel"/>
@@ -82,11 +97,11 @@
     <inertial>
         <origin xyz="0.0 0.0 0.0" rpy="0 0.0 0.0"/>
-        <mass value="0.0"/>
+        <mass value="0.3"/>
         <inertia ixx="0.0" ixy="0.0" ixz="0.0" iyy="0.0" iyz="0.0" izz="0.0"/>
     </inertial>
     <visual name="right_back_wheel_visual">
-        <origin xyz="-0.11 0.04 0.07" rpy="0 1.5707 0 "/>
-        <geometry>
-               <cylinder radius="0.05" length="0.02"/>
+        <origin xyz="0.0 0.0 0.0" rpy="0 1.5707 0 "/>
+        <geometry>
+               <cylinder radius="0.04" length="0.02"/>
         </geometry>
         <material name="">
@@ -96,12 +111,12 @@
     </visual>
     <collision>
-          <origin xyz="-0.11 0.04 0.07" rpy="0 1.5707 0 "/>
+          <origin xyz="0.0 0.0 0.0" rpy="0 1.5707 0 "/>
           <geometry>
-            <box size="0.0 0.0 0.0"/>
-        </geometry>
-    </collision>
-</link>
-<joint name="right_back_wheel_joint" type="revolute">
-    <origin xyz="-0.11 0.04 0.07" rpy="0.0 0 0"/>
+           <cylinder radius="0.04" length="0.02"/>
+        </geometry>
+    </collision>
+</link>
+<joint name="right_back_wheel_joint" type="continuous">
+    <origin xyz="-0.11 0.06 0.04" rpy="0.0 0 0"/>
     <parent link="base_plate"/>
     <child link="right_back_wheel"/>
@@ -112,11 +127,11 @@
     <inertial>
         <origin xyz="0.0 0.0 0.0" rpy="0 0.0 0.0"/>
-        <mass value="0.0"/>
+        <mass value="0.3"/>
         <inertia ixx="0.0" ixy="0.0" ixz="0.0" iyy="0.0" iyz="0.0" izz="0.0"/>
     </inertial>
     <visual name="right_front_wheel_visual">
-        <origin xyz="-0.11 0.04 -0.07" rpy="0 1.5707 0 "/>
-        <geometry>
-               <cylinder radius="0.05" length="0.02"/>
+        <origin xyz="0.0 0.0 0.0" rpy="0 1.5707 0 "/>
+        <geometry>
+               <cylinder radius="0.04" length="0.02"/>
         </geometry>
         <material name="">
@@ -126,12 +141,12 @@
     </visual>
     <collision>
-        <origin xyz="-0.11 0.04 -0.07" rpy="0 1.5707 0 "/>
-        <geometry>
-               <cylinder radius="0.05" length="0.02"/>
-        </geometry>
-    </collision>
-</link>
-<joint name="right_front_wheel_joint" type="revolute">
-    <origin xyz="-0.11 0.04 -0.07" rpy="0.0 0.0 0.0"/>
+        <origin xyz="0.0 0.0 0.0" rpy="0 1.5707 0 "/>
+        <geometry>
+               <cylinder radius="0.04" length="0.02"/>
+        </geometry>
+    </collision>
+</link>
+<joint name="right_front_wheel_joint" type="continuous">
+    <origin xyz="0.11 -0.06 0.04" rpy="0.0 0.0 0.0"/>
     <parent link="base_plate"/>
     <child link="right_front_wheel"/>
@@ -142,11 +157,11 @@
     <inertial>
         <origin xyz="0.0 0.0 0.0" rpy="0 0.0 0.0"/>
-        <mass value="0.0"/>
+        <mass value="0.4"/>
         <inertia ixx="0.0" ixy="0.0" ixz="0.0" iyy="0.0" iyz="0.0" izz="0.0"/>
     </inertial>
     <visual name="left_front_wheel_visual">
-        <origin xyz="0.11 0.04 -0.07" rpy="0 1.5707 0.0"/>
-        <geometry>
-            <cylinder radius="0.05" length="0.02"/>
+        <origin xyz="0.0 0.0 0.0" rpy="0 1.5707 0.0"/>
+        <geometry>
+            <cylinder radius="0.04" length="0.02"/>
         </geometry>
         <material name="">
@@ -156,12 +171,12 @@
     </visual>
     <collision>
-        <origin xyz="0.11 0.04 -0.07" rpy="0 1.5707 0.0"/>
-        <geometry>
-            <cylinder radius="0.05" length="0.02"/>
-        </geometry>
-    </collision>
-</link>
-<joint name="left_front_wheel_joint" type="revolute">
-    <origin xyz="0.11 0.04 -0.07" rpy="0.0 0.0 0.0"/>
+        <origin xyz="0.0 0.0 0.0" rpy="0 1.5707 0.0"/>
+        <geometry>
+            <cylinder radius="0.04" length="0.02"/>
+        </geometry>
+    </collision>
+</link>
+<joint name="left_front_wheel_joint" type="continuous">
+    <origin xyz="0.11 0.06 0.04" rpy="0.0 0.0 0.0"/>
     <parent link="base_plate"/>
     <child link="left_front_wheel"/>
@@ -169,5 +184,5 @@
     <limit lower="0.0" upper="0.0" effort="0.0" velocity="0.0"/>
 </joint>
-<link name="left_front_culom">
+<link name="left_back_culom">
     <inertial>
         <origin xyz="0.0  0.0 0.0" rpy="0 0.0 0.0"/>
@@ -176,9 +191,9 @@
     </inertial>
     <visual name="">
-        <origin xyz="0.075 .083 -0.07" rpy="0 1.5707 1.5707"/><!--.53+ .5*cylinder length-->
-        <geometry>
-            <cylinder radius="0.005" length="0.08"/>
-        </geometry>
-        <material name="left_front_culom_visual">
+        <origin xyz="0.0 0.0 0.0" rpy="0 0 1.5707"/><!--.53+ .5*cylinder length-->
+        <geometry>
+            <cylinder radius="0.005" length="0.09"/>
+        </geometry>
+        <material name="left_back_culom_visual">
             <color rgba="1.0 0.0 0.0 1.0"/>
             <texture filename=""/>
@@ -186,5 +201,5 @@
     </visual>
     <collision>
-         <origin xyz="0.075 .083 -0.07" rpy="0 1.5707 1.5707"/>
+         <origin xyz="0.0 0.0 0.0" rpy="0 1.5707 1.5707"/>
          <geometry>
              <cylinder radius="0.005" length="0.08"/>
@@ -192,15 +207,68 @@
     </collision>
 </link>
+<joint name="upper_left_back_culom_joint" type="fixed">
+    <origin xyz="-0.07 -0.1 0.1" rpy="0.0 0.0 0.0"/>
+    <parent link="base_plate"/>
+    <child link="left_back_culom"/>
+    <axis xyz="0.0 0.0 0.0"/>
+    <limit lower="0.0" upper="0.0" effort="0.0" velocity="0.0"/>
+</joint>
+<link name="right_back_colum">
+    <inertial>
+        <origin xyz="0.0 0.0 0.0" rpy="0 0.0 0.0"/>
+        <mass value="0.0"/>
+        <inertia ixx="0.0" ixy="0.0" ixz="0.0" iyy="0.0" iyz="0.0" izz="0.0"/>
+    </inertial>
+    <visual name="">
+        <origin xyz="0.0 0.0 0.0" rpy="0 0 1.5707 "/>
+        <geometry>
+            <cylinder radius="0.005" length="0.09"/>
+        </geometry>
+        <material name="right_back_colum_visual">
+            <color rgba="1.0 0.0 0.0 1.0"/>
+            <texture filename=""/>
+        </material>
+    </visual>
+    <collision>
+        <origin xyz="0.0 0.0 0.0" rpy="0 0 1.5707 "/>
+        <geometry>
+            <cylinder radius="0.005" length="0.09"/>
+        </geometry>
+    </collision>
+</link>
+<joint name="upper_right_back_culom_joint" type="fixed">
+    <origin xyz="0.07 -.1 0.1" rpy="0.0 0.0 0.0"/>
+    <parent link="base_plate"/>
+    <child link="right_back_colum"/>
+    <axis xyz="0.0 0.0 0.0"/>
+    <limit lower="0.0" upper="0.0" effort="0.0" velocity="0.0"/>
+</joint>
+<link name="left__front_colum">
+    <inertial>
+        <origin xyz="0.0 0.0 0.0" rpy="0 0.0 0.0"/>
+        <mass value="0.0"/>
+        <inertia ixx="0.0" ixy="0.0" ixz="0.0" iyy="0.0" iyz="0.0" izz="0.0"/>
+    </inertial>
+    <visual name="">
+        <origin xyz="0.0 0.0 0.0" rpy="0 0 0"/>
+        <geometry>
+            <cylinder radius="0.005" length="0.09"/>
+        </geometry>
+        <material name="left__front_colum_visual">
+            <color rgba="1.0 0.0 0.0 1.0"/>
+            <texture filename=""/>
+        </material>
+    </visual>
+    <collision>
+        <origin xyz="0.0 0.0 0.0" rpy="0 0 0"/>
+        <geometry>
+            <cylinder radius="0.005" length="0.08"/>
+        </geometry>
+    </collision>
+</link>
 <joint name="upper_left_front_culom_joint" type="fixed">
-    <origin xyz="0.075 .119 -0.07" rpy="0.0 0.0 0.0"/>
-    <parent link="base_plate"/>
-    <child link="left_front_culom"/>
-    <axis xyz="0.0 0.0 0.0"/>
-    <limit lower="0.0" upper="0.0" effort="0.0" velocity="0.0"/>
-</joint>
-<joint name="base_left_front_culom_joint" type="fixed">
-    <origin xyz="0.075 .053 -0.07" rpy="0.0 0.0 0.0"/>
-    <parent link="base_plate"/>
-    <child link="left_front_culom"/>
+    <origin xyz="0.07 .1 0.1" rpy="0.0 0.0 0.0"/>
+    <parent link="base_plate"/>
+    <child link="left__front_colum"/>
     <axis xyz="0.0 0.0 0.0"/>
     <limit lower="0.0" upper="0.0" effort="0.0" velocity="0.0"/>
@@ -213,7 +281,7 @@
     </inertial>
     <visual name="">
-        <origin xyz="-0.075 0.083 -0.07" rpy="0 1.5707 1.5707 "/>
-        <geometry>
-            <cylinder radius="0.005" length="0.08"/>
+        <origin xyz="0.0 0.0 0.0" rpy="0 0 0 "/>
+        <geometry>
+            <cylinder radius="0.005" length="0.09"/>
         </geometry>
         <material name="right_front_colum_visual">
@@ -223,5 +291,5 @@
     </visual>
     <collision>
-        <origin xyz="-0.075 0.083 -0.07" rpy="0 1.5707 1.5707 "/>
+        <origin xyz="0.0 0.0 0.0" rpy="0 0 0.0"/>
         <geometry>
             <cylinder radius="0.005" length="0.08"/>
@@ -230,88 +298,7 @@
 </link>
 <joint name="upper_right_front_culom_joint" type="fixed">
-    <origin xyz="-0.075 .119 -0.07" rpy="0.0 0.0 0.0"/>
-    <parent link="base_plate"/>
-    <child link="left_front_culom"/>
-    <axis xyz="0.0 0.0 0.0"/>
-    <limit lower="0.0" upper="0.0" effort="0.0" velocity="0.0"/>
-</joint>
-<joint name="base_right_front_culom_joint" type="fixed">
-    <origin xyz="-0.075 .053 -0.07" rpy="0.0 0.0 0.0"/>
-    <parent link="base_plate"/>
-    <child link="left_front_culom"/>
-    <axis xyz="0.0 0.0 0.0"/>
-    <limit lower="0.0" upper="0.0" effort="0.0" velocity="0.0"/>
-</joint>
-<link name="left__back_colum">
-    <inertial>
-        <origin xyz="0.0 0.0 0.0" rpy="0 0.0 0.0"/>
-        <mass value="0.0"/>
-        <inertia ixx="0.0" ixy="0.0" ixz="0.0" iyy="0.0" iyz="0.0" izz="0.0"/>
-    </inertial>
-    <visual name="">
-        <origin xyz="0.075 0.083 0.07" rpy="0 1.5707 1.5707"/>
-        <geometry>
-            <cylinder radius="0.005" length="0.08"/>
-        </geometry>
-        <material name="left__back_colum_visual">
-            <color rgba="1.0 0.0 0.0 1.0"/>
-            <texture filename=""/>
-        </material>
-    </visual>
-    <collision>
-        <origin xyz="0.075 0.083 0.07" rpy="0 1.5707 1.5707"/>
-        <geometry>
-            <cylinder radius="0.005" length="0.08"/>
-        </geometry>
-    </collision>
-</link>
-<joint name="upper_left_back_culom_joint" type="fixed">
-    <origin xyz="-0.075 .119 0.07" rpy="0.0 0.0 0.0"/>
-    <parent link="base_plate"/>
-    <child link="left_front_culom"/>
-    <axis xyz="0.0 0.0 0.0"/>
-    <limit lower="0.0" upper="0.0" effort="0.0" velocity="0.0"/>
-</joint>
-<joint name="base_left_back_culom_joint" type="fixed">
-    <origin xyz="-0.075 .053 0.07" rpy="0.0 0.0 0.0"/>
-    <parent link="base_plate"/>
-    <child link="left_front_culom"/>
-    <axis xyz="0.0 0.0 0.0"/>
-    <limit lower="0.0" upper="0.0" effort="0.0" velocity="0.0"/>
-</joint>
-<link name="right_back_colum">
-    <inertial>
-        <origin xyz="0.0 0.0 0.0" rpy="0 0.0 0.0"/>
-        <mass value="0.0"/>
-        <inertia ixx="0.0" ixy="0.0" ixz="0.0" iyy="0.0" iyz="0.0" izz="0.0"/>
-    </inertial>
-    <visual name="">
-        <origin xyz="-0.075 0.083 0.07" rpy="1.5707 1.5707 0 "/>
-        <geometry>
-            <cylinder radius="0.005" length="0.08"/>
-        </geometry>
-        <material name="right_back_colum_visual">
-            <color rgba="1.0 0.0 0.0 1.0"/>
-            <texture filename=""/>
-        </material>
-    </visual>
-    <collision>
-        <origin xyz="0.11 0.04 0.07" rpy="0 1.5707 0.0"/>
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